Commit message: add fingers support in simulation

File: franka_description/robots/hand.xacro (robot description, xacro)
@@ -17,55 +17,45 @@
       </visual>
       <collision>
-        <origin xyz="0 0 0.04" rpy="0 ${pi/2} ${pi/2}"/>
         <geometry>
-          <cylinder radius="${0.04+safety_distance}" length="0.1" />
+          <mesh filename="package://franka_description/meshes/collision/hand.stl"/>
         </geometry>
       </collision>
-      <collision>
-        <origin xyz="0 -0.05 0.04" rpy="0 0 0"/>
-        <geometry>
-          <sphere radius="${0.04+safety_distance}"  />
-        </geometry>
-      </collision>
-      <collision>
-        <origin xyz="0 0.05 0.04" rpy="0 0 0"/>
-        <geometry>
-          <sphere radius="${0.04+safety_distance}"  />
-        </geometry>
-      </collision>
-      <collision>
-        <origin xyz="0 0 0.1" rpy="0 ${pi/2} ${pi/2}"/>
-        <geometry>
-          <cylinder radius="${0.02+safety_distance}" length="0.1" />
-        </geometry>
-      </collision>
-      <collision>
-        <origin xyz="0 -0.05 0.1" rpy="0 0 0"/>
-        <geometry>
-          <sphere radius="${0.02+safety_distance}"  />
-        </geometry>
-      </collision>
-      <collision>
-        <origin xyz="0 0.05 0.1" rpy="0 0 0"/>
-        <geometry>
-          <sphere radius="${0.02+safety_distance}"  />
-        </geometry>
-      </collision>
+      <inertial>
+        <origin xyz="0 0 0" rpy="0 0 0"/>
+        <mass value="0.68"/>
+        <inertia ixx="0.1" ixy="0.0" ixz="0.0" iyy="0.1" iyz="0.0" izz="0.1"/>
+      </inertial>
     </link>
     <link name="${ns}_leftfinger">
-      <visual>
-        <geometry>
-          <mesh filename="package://franka_description/meshes/visual/finger.dae"/>
-        </geometry>
-      </visual>
-    </link>
-    <link name="${ns}_rightfinger">
-      <visual>
-        <origin xyz="0 0 0" rpy="0 0 ${pi}"/>
-        <geometry>
-          <mesh filename="package://franka_description/meshes/visual/finger.dae"/>
-        </geometry>
-      </visual>
-   </link>
+        <collision>
+          <geometry>
+            <mesh filename="package://franka_description/meshes/collision/finger.stl"/>
+          </geometry>
+        </collision>
+        <inertial>
+          <origin xyz="0 0 0" rpy="0 0 0"/>
+          <mass value="0.01"/>
+          <inertia ixx="0.1" ixy="0.0" ixz="0.0" iyy="0.1" iyz="0.0" izz="0.1"/>
+        </inertial>
+      </link>
+      <link name="${ns}_rightfinger">
+        <visual>
+          <origin xyz="0 0 0" rpy="0 0 ${pi}"/>
+          <geometry>
+            <mesh filename="package://franka_description/meshes/visual/finger.dae"/>
+          </geometry>
+        </visual>
+        <collision>
+          <origin xyz="0 0 0" rpy="0 0 ${pi}"/>
+          <geometry>
+            <mesh filename="package://franka_description/meshes/collision/finger.stl"/>
+          </geometry>
+        </collision>
+        <inertial>
+          <origin xyz="0 0 0" rpy="0 0 0"/>
+          <mass value="0.01"/>
+          <inertia ixx="0.1" ixy="0.0" ixz="0.0" iyy="0.1" iyz="0.0" izz="0.1"/>
+        </inertial>
+      </link>
     <joint name="${ns}_finger_joint1" type="prismatic">
       <parent link="${ns}_hand"/>

File: franka_description/robots/panda.gazebo.xacro (robot description, xacro)
@@ -56,4 +56,22 @@
             <mu2>0.2</mu2>
         </gazebo>
+        <!-- Hand -->
+        <gazebo reference="${robot_name}_hand">
+            <material>Gazebo/White</material>
+            <mu1>0.2</mu1>
+            <mu2>0.2</mu2>
+        </gazebo>
+        <!-- Right finger -->
+        <gazebo reference="${robot_name}_rightfinger">
+            <material>Gazebo/White</material>
+            <mu1>0.2</mu1>
+            <mu2>0.2</mu2>
+        </gazebo>
+        <!-- Link8 -->
+        <gazebo reference="${robot_name}_leftfinger">
+            <material>Gazebo/White</material>
+            <mu1>0.2</mu1>
+            <mu2>0.2</mu2>
+        </gazebo>
     </xacro:macro>
 </robot>

File: franka_description/robots/panda.transmission.xacro (robot description, xacro)
@@ -93,4 +93,28 @@
             </actuator>
         </transmission>
+        <transmission name="${robot_name}_leftfinger">
+            <type>transmission_interface/SimpleTransmission</type>
+            <joint name="${robot_name}_finger_joint1">
+                <hardwareInterface>hardware_interface/PositionJointInterface</hardwareInterface>
+                <!-- <hardwareInterface>hardware_interface/EffortJointInterface</hardwareInterface> -->
+            </joint>
+            <actuator name="${robot_name}_finger_joint1">
+                <hardwareInterface>hardware_interface/PositionJointInterface</hardwareInterface>
+                <!-- <hardwareInterface>hardware_interface/EffortJointInterface</hardwareInterface> -->
+                <mechanicalReduction>1</mechanicalReduction>
+            </actuator>
+        </transmission>
+        <transmission name="${robot_name}_rightfinger">
+            <type>transmission_interface/SimpleTransmission</type>
+            <joint name="${robot_name}_finger_joint2">
+                <hardwareInterface>hardware_interface/PositionJointInterface</hardwareInterface>
+                <!-- <hardwareInterface>hardware_interface/EffortJointInterface</hardwareInterface> -->
+            </joint>
+            <actuator name="${robot_name}_finger_joint2">
+                <hardwareInterface>hardware_interface/PositionJointInterface</hardwareInterface>
+                <!-- <hardwareInterface>hardware_interface/EffortJointInterface</hardwareInterface> -->
+                <mechanicalReduction>1</mechanicalReduction>
+            </actuator>
+        </transmission>
     </xacro:macro>
 </robot>

File: franka_description/robots/panda_arm_hand.urdf.xacro (robot description, xacro)
@@ -3,5 +3,10 @@
   <xacro:include filename="$(find franka_description)/robots/panda_arm.xacro"/>
   <xacro:include filename="$(find franka_description)/robots/hand.xacro"/>
-  <xacro:panda_arm safety_distance="0.03"/>
+  <xacro:include filename="$(find franka_description)/robots/panda.gazebo.xacro" />
+  <xacro:include filename="$(find franka_description)/robots/panda.transmission.xacro" />
+  <link name="world"/>
+  <xacro:panda_arm connected_to="world" xyz="0 0 0.86"/>
   <xacro:hand ns="panda" rpy="0 0 ${-pi/4}" connected_to="panda_link8" safety_distance="0.03"/>
+  <xacro:panda_gazebo robot_name="panda" />
+  <xacro:panda_transmission robot_name="panda" />
 </robot>

Commit message: add world link

File: franka_description/robots/hand.xacro (robot description, xacro)
@@ -28,4 +28,9 @@
     </link>
     <link name="${ns}_leftfinger">
+        <visual>
+          <geometry>
+            <mesh filename="package://franka_description/meshes/visual/finger.dae"/>
+          </geometry>
+        </visual>
         <collision>
           <geometry>
@@ -71,5 +76,4 @@
       <axis xyz="0 -1 0"/>
       <limit effort="20" lower="0.0" upper="0.04" velocity="0.2"/>
-      <mimic joint="${ns}_finger_joint1" />
     </joint>
   </xacro:macro>

File: franka_description/robots/panda_arm.urdf.xacro (robot description, xacro)
@@ -1,5 +1,22 @@
 <?xml version='1.0' encoding='utf-8'?>
 <robot xmlns:xacro="http://www.ros.org/wiki/xacro" name="panda">
-  <xacro:include filename="$(find franka_description)/robots/panda_arm.xacro" />
-  <xacro:panda_arm safety_distance="0.03"/>
+    <xacro:include filename="$(find franka_description)/robots/panda_arm.xacro" />
+    <xacro:include filename="$(find franka_description)/robots/panda.gazebo.xacro" />
+    <xacro:include filename="$(find franka_description)/robots/panda.transmission.xacro" />
+    <link name="world"/>
+    <xacro:arg name="initial_x" default="0.0"/>
+    <xacro:arg name="initial_y" default="-0.04"/>
+    <xacro:arg name="initial_z" default="0.86"/>
+    <!-- Create a fixed joint between the reference frame (world) and the robot -->
+    <joint name="world_to_arm_joint" type="fixed">
+        <parent link="world"/>
+        <child link="panda_link0"/>
+        <origin xyz="$(arg initial_x) $(arg initial_y) $(arg initial_z)" rpy="0 0.0 -1.57079632679 "/>
+    </joint>
+    <!-- Add the panda arm -->
+    <xacro:panda_arm/>
+    <!-- Add the robot properties for gazebo -->
+    <xacro:panda_gazebo robot_name="panda" />
+    <!-- Add gazebo plugin and transmission properties (linking Moveit! to Gazebo) -->
+    <xacro:panda_transmission robot_name="panda"/>
 </robot>

File: franka_description/robots/panda_arm_hand.urdf.xacro (robot description, xacro)
@@ -6,7 +6,20 @@
   <xacro:include filename="$(find franka_description)/robots/panda.transmission.xacro" />
   <link name="world"/>
-  <xacro:panda_arm connected_to="world" xyz="0 0 0.86"/>
+  <xacro:arg name="initial_x" default="0.0"/>
+  <xacro:arg name="initial_y" default="-0.04"/>
+  <xacro:arg name="initial_z" default="0.86"/>
+  <!-- Create a fixed joint between the reference frame (world) and the robot -->
+  <joint name="world_to_arm_joint" type="fixed">
+      <parent link="world"/>
+      <child link="panda_link0"/>
+      <origin xyz="$(arg initial_x) $(arg initial_y) $(arg initial_z)" rpy="0 0.0 -1.57079632679 "/>
+  </joint>
+  <!-- Add the panda arm -->
+  <xacro:panda_arm/>
+  <!-- Add robot hand -->
   <xacro:hand ns="panda" rpy="0 0 ${-pi/4}" connected_to="panda_link8" safety_distance="0.03"/>
+  <!-- Add the robot properties for gazebo -->
   <xacro:panda_gazebo robot_name="panda" />
-  <xacro:panda_transmission robot_name="panda" />
+  <!-- Add gazebo plugin and transmission properties (linking Moveit! to Gazebo) -->
+  <xacro:panda_transmission robot_name="panda"/>
 </robot>
